Commit message: for test

File: urdf/ired_robot.gazebo.xacro (robot description, xacro)
@@ -1,4 +1,4 @@
-<?xml version="1.0" ?>
-<robot name="ired_robot_gazebo" xmlns:xacro="http://ros.org/wiki/xacro">
+<?xml version="1.0"?>
+<robot name="ired_gazebo" xmlns:xacro="http://ros.org/wiki/xacro">
   <xacro:arg name="laser_visual" default="false"/>
   <xacro:arg name="imu_visual"   default="false"/>
@@ -26,22 +26,83 @@
     <material>Gazebo/FlatBlack</material>
   </gazebo>
+  <gazebo reference="caster_front_link">
+    <mu1>0.1</mu1>
+    <mu2>0.1</mu2>
+    <kp>1000000.0</kp>
+    <kd>100.0</kd>
+    <minDepth>0.001</minDepth>
+    <maxVel>1.0</maxVel>
+    <material>Gazebo/FlatBlack</material>
+  </gazebo>
+  <gazebo reference="caster_back_link">
+    <mu1>0.1</mu1>
+    <mu2>0.1</mu2>
+    <kp>1000000.0</kp>
+    <kd>100.0</kd>
+    <minDepth>0.001</minDepth>
+    <maxVel>1.0</maxVel>
+    <material>Gazebo/FlatBlack</material>
+  </gazebo>
+  <gazebo reference="imu_link">
+    <sensor type="imu" name="imu">
+      <always_on>true</always_on>
+      <visualize>$(arg imu_visual)</visualize>
+    </sensor>
+    <material>Gazebo/FlatBlack</material>
+  </gazebo>
   <gazebo>
-    <plugin filename="libgazebo_ros_diff_drive.so" name="differential_drive_controller">
-      <alwaysOn>true</alwaysOn>
-      <updateRate>10</updateRate>
+    <plugin name="differential_drive_controller" filename="libgazebo_ros_diff_drive.so">
+      <updateRate>5</updateRate>
+      <rosDebugLevel>info</rosDebugLevel>
       <leftJoint>wheel_left_joint</leftJoint>
       <rightJoint>wheel_right_joint</rightJoint>
-      <wheelSeparation>0.197</wheelSeparation>
+      <wheelSeparation>0.199</wheelSeparation>
       <wheelDiameter>0.072</wheelDiameter>
-      <torque>15</torque>
+      <wheelAcceleration>1.0</wheelAcceleration>
+      <wheelTorque>20</wheelTorque>
       <commandTopic>cmd_vel</commandTopic>
       <odometryTopic>odom</odometryTopic>
       <odometryFrame>odom</odometryFrame>
       <robotBaseFrame>base_footprint</robotBaseFrame>
+      <odometrySource>encoder</odometrySource>
+      <publishWheelTF>false</publishWheelTF> <!-- Set to false to prevent wheel TFs from being published -->
+      <publishOdom>true</publishOdom>
+      <publishOdomTF>true</publishOdomTF> <!-- Keep true if you need the odom to base_footprint TF -->
+      <publishWheelJointState>true</publishWheelJointState>
+      <legacyMode>false</legacyMode>
+      <publishTf>true</publishTf> <!-- Adjust based on your needs and plugin version -->
+    </plugin>
+  </gazebo>
+  <gazebo>
+    <plugin name="imu_plugin" filename="libgazebo_ros_imu.so">
+      <alwaysOn>true</alwaysOn>
+      <bodyName>imu_link</bodyName>
+      <frameName>imu_link</frameName>
+      <topicName>imu</topicName>
+      <serviceName>imu_service</serviceName>
+      <gaussianNoise>0.0</gaussianNoise>
+      <updateRate>0</updateRate>
+      <imu>
+        <noise>
+          <type>gaussian</type>
+          <rate>
+            <mean>0.0</mean>
+            <stddev>2e-4</stddev>
+            <bias_mean>0.0000075</bias_mean>
+            <bias_stddev>0.0000008</bias_stddev>
+          </rate>
+          <accel>
+            <mean>0.0</mean>
+            <stddev>1.7e-2</stddev>
+            <bias_mean>0.1</bias_mean>
+            <bias_stddev>0.001</bias_stddev>
+          </accel>
+        </noise>
+      </imu>
     </plugin>
   </gazebo>
   <gazebo reference="base_scan">
     <material>Gazebo/FlatBlack</material>
-    <sensor name="lidar_sensor" type="ray">
+    <sensor type="ray" name="lds_lfcd_sensor">
       <pose>0 0 0 0 0 0</pose>
       <visualize>$(arg laser_visual)</visualize>
@@ -57,6 +118,6 @@
         </scan>
         <range>
-          <min>0.12</min>
-          <max>12.0</max>
+          <min>0.25</min>
+          <max>3.5</max>
           <resolution>0.015</resolution>
         </range>
@@ -67,33 +128,9 @@
         </noise>
       </ray>
-      <plugin filename="libgazebo_ros_laser.so" name="gazebo_ros_laser_controller">
-        <topicName>/scan</topicName>
+      <plugin name="gazebo_ros_lds_lfcd_controller" filename="libgazebo_ros_laser.so">
+        <topicName>scan</topicName>
         <frameName>base_scan</frameName>
       </plugin>
     </sensor>
   </gazebo>
-  <gazebo reference="imu_link">
-    <material>Gazebo/FlatBlack</material>
-    <sensor name="imu_sensor" type="imu">
-      <always_on>true</always_on>
-      <visualize>$(arg imu_visual)</visualize>
-      <update_rate>0</update_rate>
-      <imu>
-        <angular_velocity>
-          <x>0.0</x>
-          <y>0.0</y>
-          <z>0.0</z>
-        </angular_velocity>
-        <linear_acceleration>
-          <x>0.0</x>
-          <y>0.0</y>
-          <z>0.0</z>
-        </linear_acceleration>
-      </imu>
-      <plugin filename="libgazebo_ros_imu.so" name="gazebo_ros_imu_controller">
-        <topicName>/imu</topicName>
-        <frameName>imu_link</frameName>
-      </plugin>
-    </sensor>
-  </gazebo>
 </robot>

File: urdf/ired_robot.urdf.xacro (robot description, xacro)
@@ -2,5 +2,5 @@
 <robot name="ired_robot" xmlns:xacro="http://ros.org/wiki/xacro">
   <xacro:include filename="$(find ired_simulation)/urdf/common_properties.xacro"/>
-  <xacro:include filename="$(find your_package_name)/urdf/ired_robot.gazebo.xacro" />
+  <xacro:include filename="$(find ired_simulation)/urdf/ired_robot.gazebo.xacro" />
   <!-- link -->
   <link name="base_footprint"/>
@@ -15,10 +15,16 @@
     </visual>
     <collision>
-      <origin xyz="0.0 0.05 -0.0585" rpy="1.57 0.0 3.14"/>
+      <origin xyz="0.0 0.0 0.0" rpy="0.0 0.0 0.0"/>
       <geometry>
-        <mesh filename="package://ired_simulation/meshes/Body.stl" scale="0.001 0.001 0.001"/>
+        <box size="0.25 0.18 0.143"/>
       </geometry>
-      <material name="light_black"/>
     </collision>
+    <inertial>
+      <origin xyz="0 0 0" rpy="0 0 0"/>
+      <mass value="8.2573504e-01"/>
+      <inertia ixx="2.2124416e-03" ixy="-1.2294101e-05" ixz="3.4938785e-05"
+               iyy="2.1193702e-03" iyz="-5.0120904e-06"
+               izz="2.0064271e-03" />
+    </inertial>
   </link>
   <link name="base_scan">
@@ -31,14 +37,20 @@
     </visual>
     <collision>
-      <origin xyz="0.09 -0.75 -0.143" rpy="0.0 0.0 0.0"/>
+      <origin xyz="0.015 0 -0.0065" rpy="0 0 0"/>
       <geometry>
-        <mesh filename="package://ired_simulation/meshes/LiDAR.stl" scale="0.001 0.001 0.001"/>
+        <cylinder length="0.0315" radius="0.055"/>
       </geometry>
-      <material name="dark"/>
     </collision>
+    <inertial>
+      <mass value="0.114" />
+      <origin xyz="0 0 0" />
+      <inertia ixx="0.001" ixy="0.0" ixz="0.0"
+               iyy="0.001" iyz="0.0"
+               izz="0.001" />
+    </inertial>
   </link>
   <link name="wheel_left_link">
     <visual>
-      <origin xyz="0.0 0.0 0.0" rpy="0.0 0.0 0.0"/>
+      <origin xyz="0.0 0.0 0.0" rpy="0.0 -1.57 1.57"/>
       <geometry>
         <mesh filename="package://ired_simulation/meshes/Wheel.stl" scale="0.001 0.001 0.001"/>
@@ -47,14 +59,20 @@
     </visual>
     <collision>
-      <origin xyz="0.0 0.0 0.0" rpy="0.0 0.0 0.0"/>
+      <origin xyz="0 0 0" rpy="0 0 0"/>
       <geometry>
-        <mesh filename="package://ired_simulation/meshes/Wheel.stl" scale="0.001 0.001 0.001"/>
+        <cylinder length="0.018" radius="0.033"/>
       </geometry>
-      <material name="black"/>
     </collision>
+    <inertial>
+      <origin xyz="0 0 0" />
+      <mass value="2.8498940e-02" />
+      <inertia ixx="1.1175580e-05" ixy="-4.2369783e-11" ixz="-5.9381719e-09"
+               iyy="1.1192413e-05" iyz="-1.4400107e-11"
+               izz="2.0712558e-05" />
+      </inertial>
   </link>
   <link name="wheel_right_link">
     <visual>
-      <origin xyz="0.0 0.0 0.0" rpy="0.0 0.0 0.0"/>
+      <origin xyz="0.0 0.0 0.0" rpy="0.0 1.57 1.57"/>
       <geometry>
         <mesh filename="package://ired_simulation/meshes/Wheel.stl" scale="0.001 0.001 0.001"/>
@@ -63,10 +81,46 @@
     </visual>
     <collision>
-      <origin xyz="0.0 0.0 0.0" rpy="0.0 0.0 0.0"/>
+      <origin xyz="0 0 0" rpy="0 0 0"/>
       <geometry>
-        <mesh filename="package://ired_simulation/meshes/Wheel.stl" scale="0.001 0.001 0.001"/>
+        <cylinder length="0.018" radius="0.033"/>
       </geometry>
-      <material name="black"/>
     </collision>
+    <inertial>
+      <origin xyz="0 0 0" />
+      <mass value="2.8498940e-02" />
+      <inertia ixx="1.1175580e-05" ixy="-4.2369783e-11" ixz="-5.9381719e-09"
+               iyy="1.1192413e-05" iyz="-1.4400107e-11"
+               izz="2.0712558e-05" />
+      </inertial>
+  </link>
+  <link name="caster_front_link">
+    <collision>
+      <origin xyz="0 0.005 0" rpy="0 0 0"/>
+      <geometry>
+        <box size="0.033 0.027 0.1"/>
+      </geometry>
+    </collision>
+    <inertial>
+      <origin xyz="0 0 0" />
+      <mass value="0.005" />
+      <inertia ixx="0.001" ixy="0.0" ixz="0.0"
+               iyy="0.001" iyz="0.0"
+               izz="0.001" />
+    </inertial>
+  </link>
+  <link name="caster_back_link">
+    <collision>
+      <origin xyz="0 0.005 0" rpy="0 0 0"/>
+      <geometry>
+        <box size="0.033 0.027 0.1"/>
+      </geometry>
+    </collision>
+    <inertial>
+      <origin xyz="0 0 0" />
+      <mass value="0.005" />
+      <inertia ixx="0.001" ixy="0.0" ixz="0.0"
+               iyy="0.001" iyz="0.0"
+               izz="0.001" />
+    </inertial>
   </link>
   <!-- joint -->
@@ -89,12 +143,22 @@
     <parent link="base_link"/>
     <child link="wheel_left_link"/>
-    <axis xyz="1 0 0"/>
-    <origin xyz="0.0 0.097 -0.068" rpy="0.0 0.0 1.57"/>
+    <axis xyz="0 0 1"/>
+    <origin xyz="0.0 0.097 -0.068" rpy="-1.57 0.0 0.0"/>
   </joint>
   <joint name="wheel_right_joint" type="continuous">
     <parent link="base_link"/>
     <child link="wheel_right_link"/>
-    <axis xyz="1 0 0"/>
-    <origin xyz="0.0 -0.097 -0.068" rpy="0.0 0.0 -1.57"/>
+    <axis xyz="0 0 1"/>
+    <origin xyz="0.0 -0.080 -0.068" rpy="-1.57 0.0 0.0"/>
+  </joint>
+  <joint name="caster_front_joint" type="fixed">
+    <parent link="base_link"/>
+    <child link="caster_front_link"/>
+    <origin xyz="0.11 0 -0.078" rpy="-1.57 0 0"/>
+  </joint>
+  <joint name="caster_back_joint" type="fixed">
+    <parent link="base_link"/>
+    <child link="caster_back_link"/>
+    <origin xyz="-0.11 0 -0.078" rpy="-1.57 0 0"/>
   </joint>
 </robot>
